File: hardware/packet-logger-carrier/packet-logger-carrier.kicad_pcb (KiCad board)
At the start: 2 copper layers, 86 x 58 mm, 22 parts, among them J1 RAK19003 J6, J10 RAK SPARE, J11 ESP SPARE, J12 BATT IN, J13 BATT JST-PH, J14 BATT TO RAK, J15 J15, J2 RAK19003 J7, J3 XIAO ESP32-C6, J4 microSD, J5 LID CABLE, SW1 USER BUTTON, SW2 POWER SWITCH

Commit message: hardware: set the logo lockup from the brand file, in real Archivo 900
The mark and company name were placed by eye and the wordmark was drawn in the
same crude single-stroke font used for the pin labels. Neither was accurate.

Placement now comes from handoff/logo/svg/offgrid-wordmark-horizontal.svg and
is scaled as one unit, so the proportions are the brand's:

    mark   translate(20 12) into the 200x200 beacon mark
    text   anchored x=240 y=125, size 92, letter-spacing -3
    mark height 5.4 mm -> lockup 21.0 mm wide, cap height 2.3 mm

The wordmark is now real Archivo weight 900. The variable font is instanced at
wght=900 wdth=100 with fontTools, glyph outlines are pulled, quadratic curves
flattened, and counters spliced into their outer contour with a zero-width
bridge so each letter is one simply-connected filled polygon - which both a
Gerber region and a KiCad gr_poly render correctly. Same artwork in both.

One bug worth recording: contours were first classified as outer/hole by
signed area. TrueType outers run clockwise, so that test selected the counters
and O, R and D came out as thin slivers - visible in the render as "FFG" with
fragments. Classification is now by nesting depth, which is winding-agnostic.

New gate: src/verify_wordmark.py re-renders OFFGRID through FreeType at the
same weight and compares shapes. IoU 0.94 after registration, aspect ratio
within 0.6% - the residual is antialiasing between two rasterisers, and the
overlay is essentially solid agreement. (The checker itself had the variable
axes reversed at first; this font orders them wght then wdth.)

Silkscreen gained a filled-polygon primitive, carried through silkcheck (vs
pads, holes, text, lines, accent art and the board edge), the Gerber writer as
a G36/G37 region, KiCad as a filled gr_poly, and the preview renderer.

Brand rules kept: one accent per surface - the ring is exposed copper, the
wordmark is Bone on Pitch. Clear space around the mark exceeds the 1x node
radius the han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
Other:
- board text removed: "OFFGRID"
