File: hardware/packet-logger-carrier/packet-logger-carrier.kicad_pcb (KiCad board)
At the start: 2 copper layers, 86 x 58 mm, 22 parts, among them J1 RAK19003 J6, J10 RAK SPARE, J11 ESP SPARE, J12 BATT IN, J13 BATT JST-PH, J14 BATT TO RAK, J15 J15, J2 RAK19003 J7, J3 XIAO ESP32-C6, J4 microSD, J5 LID CABLE, SW1 USER BUTTON, SW2 POWER SWITCH

Commit message: hardware: ground fill on BOTH layers, with stitching vias
We had a ground plane on the bottom only. Measured before changing anything:

    F.Cu   371 mm2 =  7.4% of the board
    B.Cu  4634 mm2 = 92.9%

That is badly unbalanced. Fabs etch and warp more evenly with copper spread
across both sides, so the top now gets a ground fill too:

    F.Cu  4280 mm2 = 85.8%
    B.Cu  4629 mm2 = 92.8%

What the fill does beyond flooding copper:

  - thermal reliefs on every GND pad on BOTH layers, so ground pins still
    solder with a normal iron
  - morphological opening at 0.30 mm, which deletes copper slivers too thin
    to etch cleanly
  - island handling: a fill region that reaches no GND pad is floating metal.
    It is either anchored with a stitching via down to the opposite plane, or
    removed. 9 stitching vias were placed; a stitch point must have room on
    BOTH layers, otherwise the via would connect to nothing.

drc.py now checks every GND pad is reached on both planes, not just B.Cu.
The Gerber writer emits both fills, and verify_gerber models both - round trip
still 0.0000 mm2 on each copper layer.

Two things found by checking rather than assuming:

  - the KiCad zone was set to island_removal_mode 1 (never remove), so KiCad
    kept 24 isolated fill islands and warned about every one. Now mode 0.
  - excluding the fill from a RECTANGLE around the brand mark left a visible
    panel of bare laminate under the soldermask - it read as a mistake in the
    render. The fill now hugs the mark's own outline at 0.35 mm, which reads
    as a deliberate halo. The router keepout box stays, so no trace crosses
    the logo.

Cross-check against KiCad's own Gerber export: both copper layers now differ
only by a thin perimeter band (~44 mm2 each) where KiCad insets its zone
slightly further from the board edge than our 0.35 mm. Both are safe.

Vias: 8 routing + 9 ground stitching = 18.

All gates pass. KiCad 10 DRC: 0 errors, 0 warnings, 0 unconnected.

Co-Authored-By: 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
Routing:
- net GND: vias 0 -> 10
- added copper zone on F.Cu, net GND
